File: G-MuzikBox.kicad_pcb (KiCad board)
At the start: 2 copper layers, 1 part, among them U1 ORANGE_PI_CM4

Commit message: update
Parts:
- added J1: USB_C_Receptacle_USB2.0_16P, Connector_USB:USB_C_Receptacle_GCT_USB4105-xx-A_16P_TopMnt_Horizontal, F.Cu at (106.7, 110.7)
Connections:
- U1 pad JP2_1: (no net) -> unconnected-(U1B-USB_OTG0_ID-PadJP2_1)
- U1 pad JP2_10: (no net) -> unconnected-(U1B-PCIE20_REFCLKP_P-PadJP2_10)
- U1 pad JP2_100: (no net) -> unconnected-(U1B-HDMI_TXDDC_SCL_PORT-PadJP2_100)
- U1 pad JP2_11: (no net) -> unconnected-(U1B-RESERVED_JP2_11-PadJP2_11)
- U1 pad JP2_12: (no net) -> unconnected-(U1B-PCIE20_REFCLKP_N-PadJP2_12)
- U1 pad JP2_13: (no net) -> unconnected-(U1B-GND_JP2_13-PadJP2_13)
- U1 pad JP2_14: (no net) -> unconnected-(U1B-GND_JP2_14-PadJP2_14)
- U1 pad JP2_15: (no net) -> unconnected-(U1B-MIPI_CSI_RX0_D0N-PadJP2_15)
- U1 pad JP2_16: (no net) -> unconnected-(U1B-PCIE20_RXP-PadJP2_16)
- U1 pad JP2_17: (no net) -> unconnected-(U1B-MIPI_CSI_RX0_D0P-PadJP2_17)
- U1 pad JP2_18: (no net) -> unconnected-(U1B-PCIE20_RXN-PadJP2_18)
- U1 pad JP2_19: (no net) -> unconnected-(U1B-GND_JP2_19-PadJP2_19)
- U1 pad JP2_2: (no net) -> unconnected-(U1B-~{PCIE20_CLKREQ_3V3_L}-PadJP2_2)
- U1 pad JP2_20: (no net) -> unconnected-(U1B-GND_JP2_20-PadJP2_20)
- U1 pad JP2_21: (no net) -> unconnected-(U1B-MIPI_CSI_RX0_D1N-PadJP2_21)
- U1 pad JP2_22: (no net) -> unconnected-(U1B-PCIE20_TXP-PadJP2_22)
- U1 pad JP2_23: (no net) -> unconnected-(U1B-MIPI_CSI_RX0_D1P-PadJP2_23)
- U1 pad JP2_24: (no net) -> unconnected-(U1B-PCIE20_TXN-PadJP2_24)
- U1 pad JP2_25: (no net) -> unconnected-(U1B-GND_JP2_25-PadJP2_25)
- U1 pad JP2_26: (no net) -> unconnected-(U1B-GND_JP2_26-PadJP2_26)
- U1 pad JP2_27: (no net) -> unconnected-(U1B-MIPI_CSI_RX_CLK0N-PadJP2_27)
- U1 pad JP2_28: (no net) -> unconnected-(U1B-MIPI_CSI_RX1_D2N-PadJP2_28)
- U1 pad JP2_29: (no net) -> unconnected-(U1B-MIPI_CSI_RX_CLK0P-PadJP2_29)
- U1 pad JP2_3: (no net) -> /USB/USB_DM
- U1 pad JP2_30: (no net) -> unconnected-(U1B-MIPI_CSI_RX1_D2P-PadJP2_30)
- U1 pad JP2_31: (no net) -> unconnected-(U1B-GND_JP2_31-PadJP2_31)
- U1 pad JP2_32: (no net) -> unconnected-(U1B-GND_JP2_32-PadJP2_32)
- U1 pad JP2_33: (no net) -> unconnected-(U1B-MIPI_CSI_RX0_D2N-PadJP2_33)
- U1 pad JP2_34: (no net) -> unconnected-(U1B-MIPI_CSI_RX1_D3N-PadJP2_34)
- U1 pad JP2_35: (no net) -> unconnected-(U1B-MIPI_CSI_RX0_D2P-PadJP2_35)
- U1 pad JP2_36: (no net) -> unconnected-(U1B-MIPI_CSI_RX1_D3P-PadJP2_36)
- U1 pad JP2_37: (no net) -> unconnected-(U1B-GND_JP2_37-PadJP2_37)
- U1 pad JP2_38: (no net) -> unconnected-(U1B-GND_JP2_38-PadJP2_38)
- U1 pad JP2_39: (no net) -> unconnected-(U1B-MIPI_CSI_RX0_D3N-PadJP2_39)
- U1 pad JP2_4: (no net) -> unconnected-(U1B-~{PCIE20_WAKE_3V3_L}-PadJP2_4)
- U1 pad JP2_40: (no net) -> unconnected-(U1B-MIPI_CSI_RX_CLK1N-PadJP2_40)
- U1 pad JP2_41: (no net) -> unconnected-(U1B-MIPI_CSI_RX0_D3P-PadJP2_41)
- U1 pad JP2_42: (no net) -> unconnected-(U1B-MIPI_CSI_RX_CLK1P-PadJP2_42)
- U1 pad JP2_43: (no net) -> unconnected-(U1B-EDP_TX_D3P-PadJP2_43)
- U1 pad JP2_44: (no net) -> unconnected-(U1B-GND_JP2_44-PadJP2_44)
- U1 pad JP2_45: (no net) -> unconnected-(U1B-EDP_SDA/I2C4_SDA_M1-PadJP2_45)
- U1 pad JP2_46: (no net) -> unconnected-(U1B-EDP_TX_D2P-PadJP2_46)
- U1 pad JP2_47: (no net) -> unconnected-(U1B-EDP_SCL/I2C4_SCL_M1-PadJP2_47)
- U1 pad JP2_48: (no net) -> unconnected-(U1B-EDP_TX_D2N-PadJP2_48)
- U1 pad JP2_49: (no net) -> unconnected-(U1B-EDP_TX_D3N-PadJP2_49)
- U1 pad JP2_5: (no net) -> /USB/USB_DP
- U1 pad JP2_50: (no net) -> unconnected-(U1B-GND_JP2_50-PadJP2_50)
- U1 pad JP2_51: (no net) -> unconnected-(U1B-HDMI_CEC_PORT-PadJP2_51)
- U1 pad JP2_52: (no net) -> unconnected-(U1B-EDP_TX_D1P-PadJP2_52)
- U1 pad JP2_53: (no net) -> unconnected-(U1B-HDMI_TX_HPD_PORT-PadJP2_53)
- U1 pad JP2_54: (no net) -> unconnected-(U1B-EDP_TX_D1N-PadJP2_54)
- U1 pad JP2_55: (no net) -> unconnected-(U1B-GND_JP2_55-PadJP2_55)
- U1 pad JP2_56: (no net) -> unconnected-(U1B-GND_JP2_56-PadJP2_56)
- U1 pad JP2_57: (no net) -> unconnected-(U1B-MIPI_DSI_TX0_D0N-PadJP2_57)
- U1 pad JP2_58: (no net) -> unconnected-(U1B-EDP_TX_D0P-PadJP2_58)
- U1 pad JP2_59: (no net) -> unconnected-(U1B-MIPI_DSI_TX0_D0P-PadJP2_59)
- U1 pad JP2_6: (no net) -> unconnected-(U1B-RESERVED_JP2_6-PadJP2_6)
- U1 pad JP2_60: (no net) -> unconnected-(U1B-EDP_TX_D0N-PadJP2_60)
- U1 pad JP2_61: (no net) -> unconnected-(U1B-GND_JP2_61-PadJP2_61)
- U1 pad JP2_62: (no net) -> unconnected-(U1B-GND_JP2_62-PadJP2_62)
- U1 pad JP2_63: (no net) -> unconnected-(U1B-MIPI_DSI_TX0_D1N-PadJP2_63)
- U1 pad JP2_64: (no net) -> unconnected-(U1B-EDP_TX_AUXP-PadJP2_64)
- U1 pad JP2_65: (no net) -> unconnected-(U1B-MIPI_DSI_TX0_D1P-PadJP2_65)
- U1 pad JP2_66: (no net) -> unconnected-(U1B-EDP_TX_AUXN-PadJP2_66)
- U1 pad JP2_67: (no net) -> unconnected-(U1B-GND_JP2_67-PadJP2_67)
- U1 pad JP2_68: (no net) -> unconnected-(U1B-GND_JP2_68-PadJP2_68)
- U1 pad JP2_69: (no net) -> unconnected-(U1B-MIPI_DSI_TX0_CLKN-PadJP2_69)
- U1 pad JP2_7: (no net) -> unconnected-(U1B-GND_JP2_7-PadJP2_7)
- U1 pad JP2_70: (no net) -> unconnected-(U1B-HDMI_TX2P_PORT-PadJP2_70)
- U1 pad JP2_71: (no net) -> unconnected-(U1B-MIPI_DSI_TX0_CLKP-PadJP2_71)
- U1 pad JP2_72: (no net) -> unconnected-(U1B-HDMI_TX2N_PORT-PadJP2_72)
- U1 pad JP2_73: (no net) -> unconnected-(U1B-GND_JP2_73-PadJP2_73)
- U1 pad JP2_74: (no net) -> unconnected-(U1B-GND_JP2_74-PadJP2_74)
- U1 pad JP2_75: (no net) -> unconnected-(U1B-MIPI_DSI_TX1_D0N-PadJP2_75)
- U1 pad JP2_76: (no net) -> unconnected-(U1B-HDMI_TX1P_PORT-PadJP2_76)
- U1 pad JP2_77: (no net) -> unconnected-(U1B-MIPI_DSI_TX1_D0P-PadJP2_77)
- U1 pad JP2_78: (no net) -> unconnected-(U1B-HDMI_TX1N_PORT-PadJP2_78)
- U1 pad JP2_79: (no net) -> unconnected-(U1B-GND_JP2_79-PadJP2_79)
- U1 pad JP2_8: (no net) -> unconnected-(U1B-GND_JP2_8-PadJP2_8)
- U1 pad JP2_80: (no net) -> unconnected-(U1B-GND_JP2_80-PadJP2_80)
- U1 pad JP2_81: (no net) -> unconnected-(U1B-MIPI_DSI_TX1_D1N-PadJP2_81)
- U1 pad JP2_82: (no net) -> unconnected-(U1B-HDMI_TX0P_PORT-PadJP2_82)
- U1 pad JP2_83: (no net) -> unconnected-(U1B-MIPI_DSI_TX1_D1P-PadJP2_83)
- U1 pad JP2_84: (no net) -> unconnected-(U1B-HDMI_TX0N_PORT-PadJP2_84)
- U1 pad JP2_85: (no net) -> unconnected-(U1B-GND_JP2_85-PadJP2_85)
- U1 pad JP2_86: (no net) -> unconnected-(U1B-GND_JP2_86-PadJP2_86)
- U1 pad JP2_87: (no net) -> unconnected-(U1B-MIPI_DSI_TX1_CLKN-PadJP2_87)
- U1 pad JP2_88: (no net) -> unconnected-(U1B-HDMI_TXCLKP_PORT-PadJP2_88)
- U1 pad JP2_89: (no net) -> unconnected-(U1B-MIPI_DSI_TX1_CLKP-PadJP2_89)
- U1 pad JP2_9: (no net) -> unconnected-(U1B-~{PCIE20_PERST_3V3_L}-PadJP2_9)
- U1 pad JP2_90: (no net) -> unconnected-(U1B-HDMI_TXCLKN_PORT-PadJP2_90)
- U1 pad JP2_91: (no net) -> unconnected-(U1B-GND_JP2_91-PadJP2_91)
- U1 pad JP2_92: (no net) -> unconnected-(U1B-GND_JP2_92-PadJP2_92)
- U1 pad JP2_93: (no net) -> unconnected-(U1B-MIPI_DSI_TX1_D2N-PadJP2_93)
- U1 pad JP2_94: (no net) -> unconnected-(U1B-MIPI_DSI_TX1_D3N-PadJP2_94)
- U1 pad JP2_95: (no net) -> unconnected-(U1B-MIPI_DSI_TX1_D2P-PadJP2_95)
- U1 pad JP2_96: (no net) -> unconnected-(U1B-MIPI_DSI_TX1_D3P-PadJP2_96)
- U1 pad JP2_97: (no net) -> unconnected-(U1B-GND_JP2_97-PadJP2_97)
- U1 pad JP2_98: (no net) -> unconnected-(U1B-GND_JP2_98-PadJP2_98)
- U1 pad JP2_99: (no net) -> unconnected-(U1B-HDMI_TXDDC_SDA_PORT-PadJP2_99)
- U1 pad JP3_1: (no net) -> unconnected-(U1C-GND_JP3_1-PadJP3_1)
- U1 pad JP3_10: (no net) -> unconnected-(U1C-MIC1_IN-PadJP3_10)
- U1 pad JP3_11: (no net) -> unconnected-(U1C-USB2_HOST2_DP-PadJP3_11)
- U1 pad JP3_12: (no net) -> unconnected-(U1C-MIC2_IN-PadJP3_12)
- U1 pad JP3_13: (no net) -> unconnected-(U1C-GND_JP3_13-PadJP3_13)
- U1 pad JP3_14: (no net) -> unconnected-(U1C-GND_JP3_14-PadJP3_14)
- U1 pad JP3_15: (no net) -> unconnected-(U1C-HP_DET_L-PadJP3_15)
- U1 pad JP3_16: (no net) -> unconnected-(U1C-USB3_HOST1_SSTXN-PadJP3_16)
- U1 pad JP3_17: (no net) -> unconnected-(U1C-GND_JP3_17-PadJP3_17)
- U1 pad JP3_18: (no net) -> unconnected-(U1C-USB3_HOST1_SSTXP-PadJP3_18)
- U1 pad JP3_19: (no net) -> unconnected-(U1C-USB3_HOST1_DM-PadJP3_19)
- U1 pad JP3_2: (no net) -> unconnected-(U1C-GND_JP3_2-PadJP3_2)
- U1 pad JP3_20: (no net) -> unconnected-(U1C-GND_JP3_20-PadJP3_20)
- U1 pad JP3_21: (no net) -> unconnected-(U1C-USB3_HOST1_DP-PadJP3_21)
- U1 pad JP3_22: (no net) -> unconnected-(U1C-USB3_HOST1_SSRXP-PadJP3_22)
- U1 pad JP3_23: (no net) -> unconnected-(U1C-GND_JP3_23-PadJP3_23)
- U1 pad JP3_24: (no net) -> unconnected-(U1C-USB3_HOST1_SSRXN-PadJP3_24)
- U1 pad JP3_3: (no net) -> unconnected-(U1C-USB2_HOST3_DM-PadJP3_3)
- U1 pad JP3_4: (no net) -> unconnected-(U1C-HPR_OUT-PadJP3_4)
- U1 pad JP3_5: (no net) -> unconnected-(U1C-USB2_HOST3_DP-PadJP3_5)
- U1 pad JP3_6: (no net) -> unconnected-(U1C-HPL_OUT-PadJP3_6)
- U1 pad JP3_7: (no net) -> unconnected-(U1C-GND_JP3_7-PadJP3_7)
- U1 pad JP3_8: (no net) -> unconnected-(U1C-HP_SNS-PadJP3_8)
- U1 pad JP3_9: (no net) -> unconnected-(U1C-USB2_HOST2_DM-PadJP3_9)
