File: G-MuzikBox.kicad_sch (KiCad schematic)
At the start: 2 parts, among them IC1 AK4458VN, U1 ORANGE_PI_CM4

Commit message: update
Parts:
- added unit 3 of U1
- added unit 2 of U1
Connections:
- new net USB/USB_DM: U1.JP2_3 (USB_OTG0_DM)
- new net USB/USB_DP: U1.JP2_5 (USB_OTG0_DP)
Other:
- added sheet USB (USB.kicad_sch)
- moved on the sheet: IC1, U1A

Commit message: dac + lpf + op-amp
Parts:
- removed IC1: AK4458VN, AK4458VN:QFN50P700X700X100-48N, symbol AK4458VN:AK4458VN
Connections:
- net I2S_SDO: now reaches U1.JP1_25 (GPIO3_D1/I2S1_SDO_M1)
- net I2S_LRCK: now reaches U1.JP1_26 (GPIO3_D0/I2S1_LRCK_M1)
- net I2S_SDI: now reaches U1.JP1_27 (GPIO3_D2/I2S1_SDI_M1)
- net I2S_SCLK: now reaches U1.JP1_49 (GPIO3_C7/I2S1_SCLK_M1)
- net I2S_MCLK: now reaches U1.JP1_50 (GPIO3_C6/I2S1_MCLK_M1)
- net DAC & opamp/SCL: now reaches U1.JP1_56 (GPIO4_B5/I2C2_SCL_M1)
- net DAC & opamp/SDA: now reaches U1.JP1_58 (GPIO4_B4/I2C2_SDA_M1)
Other:
- added sheet Amp (Amp.kicad_sch)
- added sheet DAC & opamp (DAC.kicad_sch)
- moved on the sheet: U1A, U1C

Commit message: added first 2 amps
Other:
- sheet Amp ports: added AMP_A_CLIP_OTW, AMP_A_GND, AMP_A_OUTPUTA1, AMP_A_OUTPUTA2, AMP_A_OUTPUTB1, AMP_A_OUTPUTB2, AMP_A_PVVD, AMP_A_RESET, AMP_B_CLIP_OTW, AMP_B_GND, AMP_B_OUTPUTA1, AMP_B_OUTPUTA2, AMP_B_OUTPUTB1, AMP_B_OUTPUTB2, AMP_B_PVVD, AMP_B_RESET, INPUTA, INPUTB, INPUTC, INPUTD; removed none

Commit message: this is going to be mad expensive
Other:
- sheet Amp renamed Amp1
- added sheet Amp2 (Amp2.kicad_sch)
- added sheet Power (Power.kicad_sch)
- sheet Amp1 ports: added none; removed AMP_B_OUTPUTB1, AMP_B_OUTPUTB2, INPUTD
- moved on the sheet: U1A, U1B, U1C
